File: lead/fat_bastard_lead.sch (KiCad schematic (older format))
At the start: 36 parts, among them J1 LD_12V, J2 LD_IN, J3 LD_GAIN, J4 LD_OUT, J5 HT_IN, U1 ECC83, U2 ECC83

Commit message: [lead] Add small capacitor on last gain stage's anode
The schematics has too much treble for now, and must be used with the
Tone setting between 2 and 4/10. Adding this capacitor (300-500p, tune
to taste) gives a more full-bodied sound, and enables to use the Tone
control across a broader range.
Parts:
- added C13: 500p, Capacitor_THT:C_Disc_D11.0mm_W5.0mm_P5.00mm, symbol Device:C
- C2: footprint Capacitor_THT:C_Rect_L10.0mm_W5.0mm_P5.00mm_P7.50mm -> Capacitor_THT:C_Disc_D11.0mm_W5.0mm_P5.00mm
- U1, U2: footprint Valve:Valve_ECC-83-2 -> ProjectLib:Valve_Noval-B9A_Belton-VT9-PT_Socket
Connections:
- net B+: now also C13.1
- net HT4: now also C13.2
Changed lines of the file:
@@
 Sheet 1 1
 Title "Fat Bastard"
-Date "2019-02-15"
-Rev "2"
+Date "2019-02-22"
+Rev "3"
 Comp "Arnaud Ferraris (A-wai Amplification)"
 Comment1 "Licensed under CERN OHL v.1.2"
@@
 F 0 "U1" H 4200 4475 50  0000 L CNN
 F 1 "ECC83" H 4200 4375 50  0000 L CNN
-F 2 "Valve:Valve_ECC-83-2" H 4245 4275 50  0001 C CNN
+F 2 "ProjectLib:Valve_Noval-B9A_Belton-VT9-PT_Socket" H 4245 4275 50  0001 C CNN
 F 3 "http://www.r-type.org/pdfs/ecc83.pdf" H 3975 4675 50  0001 C CNN
 	2    3975 4675
@@
 F 0 "U2" H 6878 4722 50  0000 L CNN
 F 1 "ECC83" H 6878 4629 50  0000 L CNN
-F 2 "Valve:Valve_ECC-83-2" H 6920 4275 50  0001 C CNN
+F 2 "ProjectLib:Valve_Noval-B9A_Belton-VT9-PT_Socket" H 6920 4275 50  0001 C CNN
 F 3 "http://www.r-type.org/pdfs/ecc83.pdf" H 6650 4675 50  0001 C CNN
 	2    6650 4675
@@
 F 0 "U1" H 5703 4722 50  0000 L CNN
 F 1 "ECC83" H 5703 4629 50  0000 L CNN
-F 2 "Valve:Valve_ECC-83-2" H 5745 4275 50  0001 C CNN
+F 2 "ProjectLib:Valve_Noval-B9A_Belton-VT9-PT_Socket" H 5745 4275 50  0001 C CNN
 F 3 "http://www.r-type.org/pdfs/ecc83.pdf" H 5475 4675 50  0001 C CNN
 	1    5475 4675
@@
 F 0 "U2" H 8178 4722 50  0000 L CNN
 F 1 "ECC83" H 8178 4629 50  0000 L CNN
-F 2 "Valve:Valve_ECC-83-2" H 8220 4275 50  0001 C CNN
+F 2 "ProjectLib:Valve_Noval-B9A_Belton-VT9-PT_Socket" H 8220 4275 50  0001 C CNN
 F 3 "http://www.r-type.org/pdfs/ecc83.pdf" H 7950 4675 50  0001 C CNN
 	1    7950 4675
@@
 F 0 "C2" V 4175 4225 50  0000 C CNN
 F 1 "500p" V 4475 4225 50  0000 C CNN
-F 2 "Capacitor_THT:C_Rect_L10.0mm_W5.0mm_P5.00mm_P7.50mm" H 4363 4075 50  0001 C CNN
+F 2 "Capacitor_THT:C_Disc_D11.0mm_W5.0mm_P5.00mm" H 4363 4075 50  0001 C CNN
 F 3 "~" H 4325 4225 50  0001 C CNN
 	1    4325 4225
@@
 Wire Wire Line
 	6650 3825 6650 3875
-Connection ~ 6650 3875
 Wire Wire Line
 	7950 3825 7950 3875
@@
 F 0 "U1" H 4050 1375 50  0000 L CNN
 F 1 "ECC83" H 4025 1275 50  0000 L CNN
-F 2 "Valve:Valve_ECC-83-2" H 4070 975 50  0001 C CNN
+F 2 "ProjectLib:Valve_Noval-B9A_Belton-VT9-PT_Socket" H 4070 975 50  0001 C CNN
 F 3 "http://www.r-type.org/pdfs/ecc83.pdf" H 3800 1375 50  0001 C CNN
 	3    3800 1375
@@
 F 0 "U2" H 4125 1375 50  0000 L CNN
 F 1 "ECC83" H 4050 1275 50  0000 L CNN
-F 2 "Valve:Valve_ECC-83-2" H 4795 975 50  0001 C CNN
+F 2 "ProjectLib:Valve_Noval-B9A_Belton-VT9-PT_Socket" H 4795 975 50  0001 C CNN
 F 3 "http://www.r-type.org/pdfs/ecc83.pdf" H 4525 1375 50  0001 C CNN
 	3    4525 1375
@@
 Wire Wire Line
 	4075 5425 4750 5425
+Connection ~ 6650 3875
+$Comp
+L Device:C C13
+U 1 1 5C70909A
+P 7725 4025
+AR Path="/5C70909A" Ref="C13"  Part="1"
+AR Path="/5C6397B0/5C70909A" Ref="C?"  Part="1"
+F 0 "C13" H 7475 4075 50  0000 L CNN
+F 1 "500p" H 7450 3975 50  0000 L CNN
+F 2 "Capacitor_THT:C_Disc_D11.0mm_W5.0mm_P5.00mm" H 7763 3875 50  0001 C CNN
+F 3 "~" H 7725 4025 50  0001 C CNN
+	1    7725 4025
+	1    0    0    -1
+$EndComp
+Wire Wire Line
+	7725 3875 7950 3875
+Connection ~ 7950 3875
+Wire Wire Line
+	7725 4175 7725 4225
+Wire Wire Line
+	7725 4225 7950 4225
 $EndSCHEMATC

Commit message: [lead] change footprint for C2
C2 is currently a 500p capacitor, doing heavy filtering of the low
frequencies to achieve a "modern" tone. By changing the footprint, it
can be replaced with a film capacitor (i.e. MKS4) of up to 10nF, giving
a broader range of possible tones.
Parts:
- C2: footprint Capacitor_THT:C_Disc_D11.0mm_W5.0mm_P5.00mm -> Capacitor_THT:C_Rect_L10.0mm_W5.0mm_P5.00mm_P7.50mm
Changed lines of the file:
@@
 F 0 "C2" V 4175 4225 50  0000 C CNN
 F 1 "500p" V 4475 4225 50  0000 C CNN
-F 2 "Capacitor_THT:C_Disc_D11.0mm_W5.0mm_P5.00mm" H 4363 4075 50  0001 C CNN
+F 2 "Capacitor_THT:C_Rect_L10.0mm_W5.0mm_P5.00mm_P7.50mm" H 4363 4075 50  0001 C CNN
 F 3 "~" H 4325 4225 50  0001 C CNN
 	1    4325 4225

Commit message: Add alternate component values for guitar
In its original form, this preamp could very well be used with a guitar,
providing a rather tight and modern sound.

This patch adds alternate values, designed for use with guitar,
resulting in a warmer, fuller, stoner/rock guitar tone.

Signed-off-by: Arnaud Ferraris <arnaud.ferraris@gmail.com>
Parts:
- C13: value 500p -> 360p
- C2: footprint Capacitor_THT:C_Rect_L10.0mm_W5.0mm_P5.00mm_P7.50mm -> Capacitor_THT:C_Disc_D11.0mm_W5.0mm_P5.00mm
- C5: footprint Capacitor_THT:C_Rect_L10.0mm_W3.0mm_P7.50mm_MKS4 -> Capacitor_THT:C_Rect_L13.0mm_W4.0mm_P10.00mm_FKS3_FKP3_MKS4
Other:
- note added: "For guitar, use the following\nalternate component values:\nC2 22n\nR9 39k\nC13 not fitted"
Changed lines of the file:
@@
 Sheet 1 1
 Title "Fat Bastard"
-Date "2019-02-22"
-Rev "3"
+Date "2019-05-17"
+Rev "4"
 Comp "Arnaud Ferraris (A-wai Amplification)"
 Comment1 "Licensed under CERN OHL v.1.2"
@@
 F 0 "C2" V 4175 4225 50  0000 C CNN
 F 1 "500p" V 4475 4225 50  0000 C CNN
-F 2 "Capacitor_THT:C_Rect_L10.0mm_W5.0mm_P5.00mm_P7.50mm" H 4363 4075 50  0001 C CNN
+F 2 "Capacitor_THT:C_Disc_D11.0mm_W5.0mm_P5.00mm" H 4363 4075 50  0001 C CNN
 F 3 "~" H 4325 4225 50  0001 C CNN
 	1    4325 4225
@@
 AR Path="/5C63A5EA" Ref="R3"  Part="1"
 AR Path="/5C6397B0/5C63A5EA" Ref="R?"  Part="1"
-F 0 "R3" H 4045 4072 50  0000 L CNN
-F 1 "220k" H 4045 3979 50  0000 L CNN
+F 0 "R3" H 3760 4060 50  0000 L CNN
+F 1 "220k" H 3720 3980 50  0000 L CNN
 F 2 "Resistor_THT:R_Axial_DIN0309_L9.0mm_D3.2mm_P12.70mm_Horizontal" V 3905 4025 50  0001 C CNN
 F 3 "~" H 3975 4025 50  0001 C CNN
@@
 F 0 "C5" H 6250 4075 50  0000 L CNN
 F 1 "1n" H 6250 3975 50  0000 L CNN
-F 2 "Capacitor_THT:C_Rect_L10.0mm_W3.0mm_P7.50mm_MKS4" H 6488 3875 50  0001 C CNN
+F 2 "Capacitor_THT:C_Rect_L13.0mm_W4.0mm_P10.00mm_FKS3_FKP3_MKS4" H 6488 3875 50  0001 C CNN
 F 3 "~" H 6450 4025 50  0001 C CNN
 	1    6450 4025
@@
 Wire Wire Line
 	4700 4675 4825 4675
-Text Label 4175 4225 2    50   ~ 0
+Text Label 4160 4225 2    50   ~ 0
 HT1
 Text Label 5675 4225 2    50   ~ 0
@@
 AR Path="/5C6397B0/5C70909A" Ref="C?"  Part="1"
 F 0 "C13" H 7475 4075 50  0000 L CNN
-F 1 "500p" H 7450 3975 50  0000 L CNN
+F 1 "360p" H 7450 3975 50  0000 L CNN
 F 2 "Capacitor_THT:C_Disc_D11.0mm_W5.0mm_P5.00mm" H 7763 3875 50  0001 C CNN
 F 3 "~" H 7725 4025 50  0001 C CNN
@@
 Wire Wire Line
 	7725 4225 7950 4225
+Text Notes 9670 5960 0    50   ~ 0
+For guitar, use the following\nalternate component values:\nC2    22n\nR9    39k\nC13   not fitted
+Wire Notes Line
+	9650 5520 10810 5520
+Wire Notes Line
+	10810 5520 10810 5990
+Wire Notes Line
+	10810 5990 9640 5990
+Wire Notes Line
+	9640 5990 9640 5520
 $EndSCHEMATC
